Commit message: hyq2max simplified model for test on CMAES speed in gazebo

File: urdfs/leg/leg.urdf.xacro (robot description, xacro)
@@ -63,5 +63,6 @@
 				<origin xyz="0 -0.046 0" rpy="0 ${-PI/2} ${-PI/2}"/>
 				<geometry>
-					<mesh filename="package://hyq2max_description/meshes/leg/hipassembly.dae" scale="1 1 1"/>
+					<!-- <mesh filename="package://hyq2max_description/meshes/leg/hipassembly.dae" scale="1 1 1"/> -->
+				<cylinder length="0.117" radius="0.0444"/>
 				</geometry>
 			</visual>
@@ -69,5 +70,6 @@
 				<origin xyz="0 -0.046 0" rpy="0 ${-PI/2} ${-PI/2}"/>
 				<geometry>
-					<mesh filename="package://hyq2max_description/meshes/leg/hipassembly.dae" scale="1 1 1"/>
+					<!-- <mesh filename="package://hyq2max_description/meshes/leg/hipassembly.dae" scale="1 1 1"/> -->
+				<cylinder length="0.117" radius="0.0444"/>
 				</geometry>
 			</collision>
@@ -82,13 +84,19 @@
 			</inertial>
 			<visual>
-				<origin xyz="0 0 ${-0.03*reflect_left}" rpy="${(1-reflect_left)*PI/2} 0 0"/>
+				<!-- <origin xyz="0 0 ${-0.03*reflect_left}" rpy="${(1-reflect_left)*PI/2} 0 0"/> -->
+				<origin xyz="0.180 0 0" rpy="0 0 0"/>
 				<geometry>
-					<mesh filename="package://hyq2max_description/meshes/leg/upperleg.dae" scale="1 1 1"/>
+					<!-- <mesh filename="package://hyq2max_description/meshes/leg/upperleg.dae" scale="1 1 1"/> -->
+				<box size="0.360 0.116 0.07"/>
+				<!-- <cylinder length="0.360" radius="0.07"/> -->
 				</geometry>
 			</visual>
 			<collision>
-				<origin xyz="0 0 ${-0.03*reflect_left}" rpy="${(1-reflect_left)*PI/2} 0 0"/>
+				<!-- <origin xyz="0 0 ${-0.03*reflect_left}" rpy="${(1-reflect_left)*PI/2} 0 0"/> -->
+				<origin xyz="0.180 0 0" rpy="0 0 0"/>
 				<geometry>
-					<mesh filename="package://hyq2max_description/meshes/leg/upperleg.dae" scale="1 1 1"/>
+					<!-- <mesh filename="package://hyq2max_description/meshes/leg/upperleg.dae" scale="1 1 1"/> -->
+				<box size="0.360 0.116 0.07"/>
+				<!-- <cylinder length="0.360" radius="0.07"/> -->
 				</geometry>
 			</collision>
@@ -103,14 +111,18 @@
 			</inertial>
 			<visual>
-				<origin xyz="0 0 0" rpy="${(1-reflect_front)*PI/2} 0 ${PI-reflect_front*knee_offset_angle*PI/180}"/>
+				<!-- <origin xyz="0 0 0" rpy="${(1-reflect_front)*PI/2} 1.57 ${PI-reflect_front*knee_offset_angle*PI/180}"/> -->
+				<origin xyz="0.190 0 0" rpy="0 1.57 0"/>
 				<geometry>
-					<mesh filename="package://hyq2max_description/meshes/leg/lowerleg.dae" scale="1 1 1"/>
+<!--			<mesh filename="package://hyq2max_description/meshes/leg/lowerleg.dae" scale="1 1 1"/> -->
+				<cylinder length="0.380" radius="0.02"/>
 				</geometry>
 				<material name="white"/>
 			</visual>
 			<collision>
-				<origin xyz="0 0 0" rpy="${(1-reflect_front)*PI/2} 0 ${PI-reflect_front*knee_offset_angle*PI/180}"/>
+				<!-- <origin xyz="0 0 0" rpy="${(1-reflect_front)*PI/2} 1.57 ${PI-reflect_front*knee_offset_angle*PI/180}"/> -->
+				<origin xyz="0.190 0 0" rpy="0 1.57 0"/>
 				<geometry>
-					<mesh filename="package://hyq2max_description/meshes/leg/lowerleg.dae" scale="1 1 1"/>
+<!--			<mesh filename="package://hyq2max_description/meshes/leg/lowerleg.dae" scale="1 1 1"/> -->
+				<cylinder length="0.380" radius="0.02"/>
 				</geometry>
 			</collision>
@@ -123,10 +135,10 @@
 				<inertia ixx="0.0" iyy="0.0" izz="0.0" ixy="0.0" ixz="0.0" iyz="0.0"/>
 			</inertial>
-			<!--<visual>
+			<visual>
 				<origin xyz="0.0 0.0 0.0" rpy="0.0 0.0 0.0"/>
 				<geometry>
 					<sphere radius="0.021"/>
 				</geometry>
-			</visual>-->
+			</visual>
 			<collision>
 				<origin xyz="0 0 0" rpy="0 0 0"/>

File: urdfs/trunk/trunk.urdf.xacro (robot description, xacro)
@@ -30,13 +30,17 @@
 			</inertial>
 			<visual>
-				<origin xyz="0 0 0" rpy="${PI/2} 0 ${PI/2}" />
+				<!-- <origin xyz="0 0 0" rpy="${PI/2} 0 ${PI/2}" /> -->
+				<origin xyz="0 0 0" rpy="0 0 0" />
 				<geometry>
-					<mesh filename="package://hyq2max_description/meshes/trunk/trunk.dae" scale="${trunkScale_width} 1 ${trunkScale_length}"/>
+<!-- 					<mesh filename="package://hyq2max_description/meshes/trunk/trunk.dae" scale="${trunkScale_width} 1 ${trunkScale_length}"/> -->
+				 <box size="1.306 0.400 0.318"/>
 				</geometry>
 			</visual>
 			<collision>
-				<origin xyz="0 0 0" rpy="${PI/2} 0 ${PI/2}" />
+				<!-- <origin xyz="0 0 0" rpy="${PI/2} 0 ${PI/2}" /> -->
+				<origin xyz="0 0 0" rpy="0 0 0" />
 				<geometry>
-					<mesh filename="package://hyq2max_description/meshes/trunk/trunk.dae" scale="${trunkScale_width} 1 ${trunkScale_length}"/>
+<!-- 					<mesh filename="package://hyq2max_description/meshes/trunk/trunk.dae" scale="${trunkScale_width} 1 ${trunkScale_length}"/> -->
+				<box size="1.306 0.400 0.318"/>
 				</geometry>
 			</collision>

Commit message: hyqReal mockup based on hyq2max

File: urdfs/leg/leg.urdf.xacro (robot description, xacro)
@@ -84,18 +84,18 @@
 			</inertial>
 			<visual>
-				<!-- <origin xyz="0 0 ${-0.03*reflect_left}" rpy="${(1-reflect_left)*PI/2} 0 0"/> -->
-				<origin xyz="0.180 0 0" rpy="0 0 0"/>
+				<origin xyz="0 0 ${-0.03*reflect_left}" rpy="${(1-reflect_left)*PI/2} 0 0"/>
+				<!-- <origin xyz="0.180 0 0" rpy="0 0 0"/> -->
 				<geometry>
-					<!-- <mesh filename="package://hyq2max_description/meshes/leg/upperleg.dae" scale="1 1 1"/> -->
-				<box size="0.360 0.116 0.07"/>
+					<mesh filename="package://hyq2max_description/meshes/leg/upperleg.dae" scale="1 1 1"/>
+				<!-- <box size="0.360 0.116 0.07"/> -->
 				<!-- <cylinder length="0.360" radius="0.07"/> -->
 				</geometry>
 			</visual>
 			<collision>
-				<!-- <origin xyz="0 0 ${-0.03*reflect_left}" rpy="${(1-reflect_left)*PI/2} 0 0"/> -->
-				<origin xyz="0.180 0 0" rpy="0 0 0"/>
+				<origin xyz="0 0 ${-0.03*reflect_left}" rpy="${(1-reflect_left)*PI/2} 0 0"/>
+				<!-- <origin xyz="0.180 0 0" rpy="0 0 0"/> -->
 				<geometry>
-					<!-- <mesh filename="package://hyq2max_description/meshes/leg/upperleg.dae" scale="1 1 1"/> -->
-				<box size="0.360 0.116 0.07"/>
+					<mesh filename="package://hyq2max_description/meshes/leg/upperleg.dae" scale="1 1 1"/>
+				<!-- <box size="0.360 0.116 0.07"/> -->
 				<!-- <cylinder length="0.360" radius="0.07"/> -->
 				</geometry>
@@ -111,18 +111,14 @@
 			</inertial>
 			<visual>
-				<!-- <origin xyz="0 0 0" rpy="${(1-reflect_front)*PI/2} 1.57 ${PI-reflect_front*knee_offset_angle*PI/180}"/> -->
-				<origin xyz="0.190 0 0" rpy="0 1.57 0"/>
+				<origin xyz="0 0 0" rpy="${(1-reflect_front)*PI/2} 0 ${PI-reflect_front*knee_offset_angle*PI/180}"/>
 				<geometry>
-<!--			<mesh filename="package://hyq2max_description/meshes/leg/lowerleg.dae" scale="1 1 1"/> -->
-				<cylinder length="0.380" radius="0.02"/>
+					<mesh filename="package://hyq2max_description/meshes/leg/lowerleg.dae" scale="1 1 1"/>
 				</geometry>
 				<material name="white"/>
 			</visual>
 			<collision>
-				<!-- <origin xyz="0 0 0" rpy="${(1-reflect_front)*PI/2} 1.57 ${PI-reflect_front*knee_offset_angle*PI/180}"/> -->
-				<origin xyz="0.190 0 0" rpy="0 1.57 0"/>
+				<origin xyz="0 0 0" rpy="${(1-reflect_front)*PI/2} 0 ${PI-reflect_front*knee_offset_angle*PI/180}"/>
 				<geometry>
-<!--			<mesh filename="package://hyq2max_description/meshes/leg/lowerleg.dae" scale="1 1 1"/> -->
-				<cylinder length="0.380" radius="0.02"/>
+					<mesh filename="package://hyq2max_description/meshes/leg/lowerleg.dae" scale="1 1 1"/>
 				</geometry>
 			</collision>

File: urdfs/trunk/trunk.urdf.xacro (robot description, xacro)
@@ -30,16 +30,16 @@
 			</inertial>
 			<visual>
-				<origin xyz="0 0 0" rpy="${PI/2} 0 ${PI/2}" />
+				<origin xyz="0 0 0" rpy="0 0 ${PI}" />
 				<!-- <origin xyz="0 0 0" rpy="0 0 0" /> -->
 				<geometry>
- 					<mesh filename="package://hyq2max_description/meshes/trunk/trunk.dae" scale="${trunkScale_width} 1 ${trunkScale_length}"/>
+ 					<mesh filename="package://hyq2max_description/meshes/trunk/trunk.dae" scale="0.001 0.001 0.001"/>
 				 <!-- <box size="1.306 0.400 0.318"/>  -->
 				</geometry>
 			</visual>
 			<collision>
-				<origin xyz="0 0 0" rpy="${PI/2} 0 ${PI/2}" />
+				<origin xyz="0 0 0" rpy="0 0 ${PI}" />
 				<!-- <origin xyz="0 0 0" rpy="0 0 0" /> -->
 				<geometry>
-					<mesh filename="package://hyq2max_description/meshes/trunk/trunk.dae" scale="${trunkScale_width} 1 ${trunkScale_length}"/>
+					<mesh filename="package://hyq2max_description/meshes/trunk/trunk.dae" scale="0.001 0.001 0.001"/>
 				<!-- <box size="1.306 0.400 0.318"/>  -->
 				</geometry>

File: urdfs/trunk/trunk_model.urdf.xacro (robot description, xacro)
@@ -30,13 +30,13 @@
 			</inertial>
 			<visual>
-				<origin xyz="0 0 0" rpy="${PI/2} 0 ${PI/2}" />
+				<origin xyz="0 0 0" rpy="0 0 ${PI}" />
 				<geometry>
-					<mesh filename="package://hyq2max_description/meshes/trunk/trunk.dae" scale="${trunkScale_width} 1 ${trunkScale_length}"/>
+					<mesh filename="package://hyq2max_description/meshes/trunk/trunk.dae" scale="0.001 0.001 0.001"/>
 				</geometry>
 			</visual>
 			<collision>
-				<origin xyz="0 0 0" rpy="${PI/2} 0 ${PI/2}" />
+				<origin xyz="0 0 0" rpy="0 0 ${PI}" />
 				<geometry>
-					<mesh filename="package://hyq2max_description/meshes/trunk/trunk.dae" scale="${trunkScale_width} 1 ${trunkScale_length}"/>
+					<mesh filename="package://hyq2max_description/meshes/trunk/trunk.dae" scale="0.001 0.001 0.001"/>
 				</geometry>
 			</collision>
