Commit message: Merge branch 'master' into AR_hyq2max
Conflicts:
	robcogen/hyq2max.kindsl

File: urdfs/trunk/trunk.urdf.xacro (robot description, xacro)
@@ -30,17 +30,17 @@
 			</inertial>
 			<visual>
-				<!-- <origin xyz="0 0 0" rpy="${PI/2} 0 ${PI/2}" /> -->
-				<origin xyz="0 0 0" rpy="0 0 0" />
+				<origin xyz="0 0 0" rpy="${PI/2} 0 ${PI/2}" />
+				<!-- <origin xyz="0 0 0" rpy="0 0 0" /> -->
 				<geometry>
-<!-- 					<mesh filename="package://hyq2max_description/meshes/trunk/trunk.dae" scale="${trunkScale_width} 1 ${trunkScale_length}"/> -->
-				 <box size="1.306 0.400 0.318"/>
+ 					<mesh filename="package://hyq2max_description/meshes/trunk/trunk.dae" scale="${trunkScale_width} 1 ${trunkScale_length}"/>
+				 <!-- <box size="1.306 0.400 0.318"/>  -->
 				</geometry>
 			</visual>
 			<collision>
-				<!-- <origin xyz="0 0 0" rpy="${PI/2} 0 ${PI/2}" /> -->
-				<origin xyz="0 0 0" rpy="0 0 0" />
+				<origin xyz="0 0 0" rpy="${PI/2} 0 ${PI/2}" />
+				<!-- <origin xyz="0 0 0" rpy="0 0 0" /> -->
 				<geometry>
-<!-- 					<mesh filename="package://hyq2max_description/meshes/trunk/trunk.dae" scale="${trunkScale_width} 1 ${trunkScale_length}"/> -->
-				<box size="1.306 0.400 0.318"/>
+					<mesh filename="package://hyq2max_description/meshes/trunk/trunk.dae" scale="${trunkScale_width} 1 ${trunkScale_length}"/>
+				<!-- <box size="1.306 0.400 0.318"/>  -->
 				</geometry>
 			</collision>

Commit message: [xacro aligned with dae]

File: urdfs/trunk/trunk.urdf.xacro (robot description, xacro)
@@ -30,16 +30,16 @@
 			</inertial>
 			<visual>
-				<origin xyz="0 0 0" rpy="0 0 ${PI}" />
+				<origin xyz="0 0 0" rpy="${PI/2} 0 ${PI/2}" />
 				<!-- <origin xyz="0 0 0" rpy="0 0 0" /> -->
 				<geometry>
- 					<mesh filename="package://hyq2max_description/meshes/trunk/trunk.dae" scale="0.001 0.001 0.001"/>
+ 					<mesh filename="package://hyq2max_description/meshes/trunk/trunk.dae" scale="${trunkScale_width} 1 ${trunkScale_length}"/>
 				 <!-- <box size="1.306 0.400 0.318"/>  -->
 				</geometry>
 			</visual>
 			<collision>
-				<origin xyz="0 0 0" rpy="0 0 ${PI}" />
+				<origin xyz="0 0 0" rpy="${PI/2} 0 ${PI/2}" />
 				<!-- <origin xyz="0 0 0" rpy="0 0 0" /> -->
 				<geometry>
-					<mesh filename="package://hyq2max_description/meshes/trunk/trunk.dae" scale="0.001 0.001 0.001"/>
+					<mesh filename="package://hyq2max_description/meshes/trunk/trunk.dae" scale="${trunkScale_width} 1 ${trunkScale_length}"/>
 				<!-- <box size="1.306 0.400 0.318"/>  -->
 				</geometry>

File: urdfs/trunk/trunk_model.urdf.xacro (robot description, xacro)
@@ -30,13 +30,13 @@
 			</inertial>
 			<visual>
-				<origin xyz="0 0 0" rpy="0 0 ${PI}" />
+				<origin xyz="0 0 0" rpy="${PI/2} 0 ${PI/2}" />
 				<geometry>
-					<mesh filename="package://hyq2max_description/meshes/trunk/trunk.dae" scale="0.001 0.001 0.001"/>
+					<mesh filename="package://hyq2max_description/meshes/trunk/trunk.dae" scale="${trunkScale_width} 1 ${trunkScale_length}"/>
 				</geometry>
 			</visual>
 			<collision>
-				<origin xyz="0 0 0" rpy="0 0 ${PI}" />
+				<origin xyz="0 0 0" rpy="${PI/2} 0 ${PI/2}" />
 				<geometry>
-					<mesh filename="package://hyq2max_description/meshes/trunk/trunk.dae" scale="0.001 0.001 0.001"/>
+					<mesh filename="package://hyq2max_description/meshes/trunk/trunk.dae" scale="${trunkScale_width} 1 ${trunkScale_length}"/>
 				</geometry>
 			</collision>
