Commit message: including soft and hard shell dae, incorporated trunk params from CAD

File: urdfs/common.xacro (robot description, xacro)
@@ -5,5 +5,5 @@
 	<property name="d_lr" value="0.414"/>
 	<property name="d_fh" value="0.747"/>
-	<property name="haa_lr" value="0.194"/>
+	<property name="haa_lr" value="0.278"/>
 	<!-- 0.194  0.34125 -->
 	<property name="haa_fh" value="0.887"/>
@@ -18,14 +18,14 @@
 	<!-- Inertial values -->
 	<!-- Trunk with hydraulic system -->
-	<property name="xcom_trunk" value="0.060663"/>
-	<property name="ycom_trunk" value="0.000598"/>
-	<property name="zcom_trunk" value="-0.007592"/>
-	<property name="m_trunk" value="39.71"/>
-	<property name="ixx_trunk" value="0.3020795"/>
-	<property name="iyy_trunk" value="4.751448"/>
-	<property name="izz_trunk" value="4.82415"/>
-	<property name="ixy_trunk" value="-0.0050854"/>
-	<property name="ixz_trunk" value=" 0.0046576"/>
-	<property name="iyz_trunk" value="-0.0017613"/>
+	<property name="xcom_trunk" value="-0.503079700"/>
+	<property name="ycom_trunk" value="0.000012738"/>
+	<property name="zcom_trunk" value="-0.105401681219"/>
+	<property name="m_trunk" value="44.143"/>
+	<property name="ixx_trunk" value="0.433864"/>
+	<property name="iyy_trunk" value="3.128618"/>
+	<property name="izz_trunk" value="3.133731"/>
+	<property name="ixy_trunk" value="-0.000000214278701"/>
+	<property name="ixz_trunk" value="-0.003014101103917"/>
+	<property name="iyz_trunk" value=" 0.000000003318123"/>
 	<!-- Hip assembly -->
 	<property name="xcom_hipassembly" value="-0.000605"/>

File: urdfs/trunk/trunk.urdf.xacro (robot description, xacro)
@@ -30,5 +30,5 @@
 			</inertial>
 			<visual>
-				<origin xyz="0 0 0" rpy="0 0 ${PI}" />
+				<origin xyz="0 0 0.025" rpy="0 0 ${PI}" />
 				<!-- <origin xyz="0 0 0" rpy="0 0 0" /> -->
 				<geometry>
@@ -38,5 +38,5 @@
 			</visual>
 			<collision>
-				<origin xyz="0 0 0" rpy="0 0 ${PI}" />
+				<origin xyz="0 0 0.025" rpy="0 0 ${PI}" />
 				<!-- <origin xyz="0 0 0" rpy="0 0 0" /> -->
 				<geometry>

Commit message: params as in hyqreal dae

File: urdfs/common.xacro (robot description, xacro)
@@ -18,6 +18,6 @@
 	<!-- Inertial values -->
 	<!-- Trunk with hydraulic system -->
-	<property name="xcom_trunk" value="-0.503079700"/>
-	<property name="ycom_trunk" value="0.000012738"/>
+	<property name="xcom_trunk" value="-0.000503079700"/>
+	<property name="ycom_trunk" value=" 0.000000012738"/>
 	<property name="zcom_trunk" value="-0.105401681219"/>
 	<property name="m_trunk" value="44.143"/>

File: urdfs/trunk/trunk.urdf.xacro (robot description, xacro)
@@ -30,5 +30,5 @@
 			</inertial>
 			<visual>
-				<origin xyz="0 0 0.025" rpy="0 0 ${PI}" />
+				<origin xyz="0 0 0.0" rpy="0 0 ${PI}" />
 				<!-- <origin xyz="0 0 0" rpy="0 0 0" /> -->
 				<geometry>
@@ -38,5 +38,5 @@
 			</visual>
 			<collision>
-				<origin xyz="0 0 0.025" rpy="0 0 ${PI}" />
+				<origin xyz="0 0 0.0" rpy="0 0 ${PI}" />
 				<!-- <origin xyz="0 0 0" rpy="0 0 0" /> -->
 				<geometry>

Commit message: cosmetics

File: urdfs/common.xacro (robot description, xacro)
@@ -21,4 +21,5 @@
 	<property name="ycom_trunk" value=" 0.000000012738"/>
 	<property name="zcom_trunk" value="-0.105401681219"/>
+	<!-- <property name="zcom_trunk" value="-0.050"/> -->
 	<property name="m_trunk" value="44.143"/>
 	<property name="ixx_trunk" value="0.433864"/>

File: urdfs/trunk/trunk.urdf.xacro (robot description, xacro)
@@ -30,5 +30,5 @@
 			</inertial>
 			<visual>
-				<origin xyz="0 0 0.0" rpy="0 0 ${PI}" />
+				<origin xyz="0 0 0" rpy="0 0 ${PI}" />
 				<!-- <origin xyz="0 0 0" rpy="0 0 0" /> -->
 				<geometry>
@@ -38,5 +38,5 @@
 			</visual>
 			<collision>
-				<origin xyz="0 0 0.0" rpy="0 0 ${PI}" />
+				<origin xyz="0 0 0" rpy="0 0 ${PI}" />
 				<!-- <origin xyz="0 0 0" rpy="0 0 0" /> -->
 				<geometry>
